File: KiCAD/Projects/ESP8266_adapter/ESP8266_adapter.kicad_pcb (KiCad board)
At the start: 2 copper layers, 13 parts, among them P1 PWR, P2 CONN_LEFT, P3 CONN_RIGHT, P4 UART_PROG, P5 PWR, SW1 RST_SWITCH, U1 NCP1117ST33T3G, U2 ESP-12E

Commit message: Initial commit
Parts:
- added P6: PWR, Pin_Headers:Pin_Header_Straight_1x02_Pitch2.54mm, F.Cu at (65.3, 68.5)
- C3: footprint Capacitors_THT:C_Disc_D7.5mm_W5.0mm_P10.00mm -> Capacitors_ThroughHole:C_Disc_D7.0mm_W2.5mm_P5.00mm
- P1: footprint Connectors_Phoenix:PhoenixContact_MSTBVA-G_02x5.00mm_Vertical -> Connectors_Phoenix:PhoenixContact_MCV-G_02x5.08mm_Vertical
- U1: value NCP1117ST33T3G -> NCP1117DT33G_MountingTab
- moved SW1 61.2 mm to (32.8, 64.8), turned to 270 degrees
- moved R1 52.7 mm to (24.1, 42.2), turned to 90 degrees
- moved P4 50.5 mm to (67.8, 65.2), turned to 270 degrees
- moved C3 46.9 mm to (39.3, 70.8), turned to 90 degrees
- moved R2 37.1 mm to (36.3, 61.5), turned to 315 degrees
- moved P5 13.2 mm to (32.7, 76.6), turned to 90 degrees
- moved P1 12.4 mm to (58.1, 75.0), turned to 0 degrees
- moved U1 12.0 mm to (47.5, 63.3), turned to 90 degrees
- moved C1 10.1 mm to (43.1, 74.0), turned to 270 degrees
- moved C2 8.52 mm to (51.6, 75.2), turned to 180 degrees
- moved P3 3.60 mm to (63.0, 32.3)
- moved P2 2.71 mm to (27.4, 32.3)
- moved U2 2.09 mm to (39.5, 31.3)
Connections:
- C1 pad 2: +5V -> GND
- C2 pad 2: +5V -> GND
- C3 pad 1: +5V -> GND
- P1 pad 1: +5V -> GND
- P3 pad 15: +5V -> GND
- P3 pad 16: +5V -> GND
- P4 pad 1: +5V -> /3V3
- P4 pad 2: Net-(P4-Pad2) -> /5V
- P4 pad 5: +5V -> GND
- P5 pad 1: +5V -> GND
- SW1 pad 2: +5V -> GND
- SW1 pad 4: +5V -> GND
- U1 pad 1: +5V -> GND
- U1 pad 4: (no net) -> +3V3
- U2 pad 9: +5V -> GND
Routing:
- net +3V3: track 0.00 -> 84.6 mm
- net RESET: track 0.00 -> 67.0 mm
- net Tx: track 0.00 -> 56.9 mm
- net Rx: track 0.00 -> 54.1 mm
- net GPIO9: track 0.00 -> 25.4 mm
- net GPIO10: track 0.00 -> 25.3 mm
- net MISO: track 0.00 -> 21.8 mm
- net MOSI: track 0.00 -> 21.7 mm
- net GND: track 0.00 -> 19.0 mm
- net EN: track 0.00 -> 18.5 mm
- net SCLK: track 0.00 -> 18.2 mm
- net CS: track 0.00 -> 18.1 mm
- net GPIO13: track 0.00 -> 13.8 mm
- net GPIO15: track 0.00 -> 13.8 mm
- net GPIO12: track 0.00 -> 13.6 mm
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- added copper zone on F.Cu, net +3V3
- added copper zone on F.Cu, net GND
Other:
- board outline added: 52.7 x 51.4 mm

Commit message: Update with minor modifications
Other:
- board text added: "ESP12F Adapter ABN 2017"
Changed lines of the file:
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@@
     (links 70)
     (no_connects 0)
-    (area 17.704999 27.864999 86.435001 81.355001)
+    (area 20.244999 22.324999 73.100001 81.355001)
     (thickness 1.6)
-    (drawings 6)
-    (tracks 184)
+    (drawings 7)
+    (tracks 183)
     (zones 0)
     (modules 14)
@@
     (user_trace_width 2.25)
     (trace_clearance 0.2)
-    (zone_clearance 0.7)
-    (zone_45_only no)
+    (zone_clearance 0.6)
+    (zone_45_only yes)
     (trace_min 0.2)
     (segment_width 0.2)
@@
     (visible_elements 7FFDFFFF)
     (pcbplotparams
-      (layerselection 0x00030_ffffffff)
+      (layerselection 0x00000_7fffffff)
       (usegerberextensions false)
       (excludeedgelayer true)
@@
       (padsonsilk false)
       (subtractmaskfromsilk false)
-      (outputformat 1)
+      (outputformat 4)
       (mirror false)
       (drillshape 1)
@@
     )
   )
+  (gr_text "ESP12F Adapter\nABN 2017" (at 46.5 56.75) (layer F.Cu)
+    (effects (font (size 0.6 0.6) (thickness 0.1)))
+  )
   (gr_line (start 73.025 81.28) (end 71.12 81.28) (angle 90) (layer Edge.Cuts) (width 0.15))
   (gr_line (start 73.025 29.845) (end 73.025 81.28) (angle 90) (layer Edge.Cuts) (width 0.15))
@@
   (segment (start 43.0784 71.3994) (end 44.0278 70.45) (width 1.25) (layer F.Cu) (net 1))
   (segment (start 43.0684 74.0002) (end 43.0784 73.9902) (width 0.25) (layer F.Cu) (net 1) (status 30))
-  (segment (start 29.93 50.1) (end 27.39 50.1) (width 1.25) (layer F.Cu) (net 2) (status C00000))
+  (segment (start 29.93 50.1) (end 33.15 50.1) (width 1.25) (layer F.Cu) (net 2) (status 400000))
+  (segment (start 33.15 50.1) (end 37.95 45.3) (width 1.25) (layer F.Cu) (net 2) (status 800000))
+  (segment (start 37.95 45.3) (end 39.45 45.3) (width 0.25) (layer F.Cu) (net 2) (status C00000))
+  (segment (start 29.93 50.1) (end 27.39 50.1) (width 1.25) (layer F.Cu) (net 2))
   (segment (start 25.6525 50.1) (end 24.13 50.1) (width 1.25) (layer F.Cu) (net 2))
   (segment (start 24.13 50.1) (end 24.13 50.165) (width 1.25) (layer F.Cu) (net 2))
@@
   (segment (start 25.535786 60.135786) (end 25.4 60.135786) (width 1.25) (layer F.Cu) (net 2))
   (segment (start 25.4 60.135786) (end 34.885786 60.135786) (width 1.25) (layer F.Cu) (net 2))
-  (segment (start 29.93 50.1) (end 32.8 50.1) (width 1) (layer F.Cu) (net 2))
-  (segment (start 32.8 50.1) (end 34.8 48.1) (width 1) (layer F.Cu) (net 2))
-  (segment (start 34.8 48.1) (end 36.65 48.1) (width 1) (layer F.Cu) (net 2))
-  (segment (start 36.65 48.1) (end 39.45 45.3) (width 1) (layer F.Cu) (net 2))
   (segment (start 24.13 40.2148) (end 24.13 38.2905) (width 1.25) (layer F.Cu) (net 3))
   (segment (start 25.0205 37.4) (end 27.39 37.4) (width 1.25) (layer F.Cu) (net 3))
@@
   (segment (start 32.85 34.85) (end 34.4 33.3) (width 1) (layer F.Cu) (net 12))
   (segment (start 34.4 33.3) (end 39.45 33.3) (width 1) (layer F.Cu) (net 12))
-  (segment (start 62.67 65.25) (end 62.67 64.2665) (width 0.75) (layer F.Cu) (net 13) (status 400000))
+  (segment (start 62.67 65.25) (end 62.67 64.2665) (width 0.75) (layer F.Cu) (net 13))
   (segment (start 69.912 32.32) (end 71.3105 33.7185) (width 0.75) (layer F.Cu) (net 13))
   (segment (start 71.3105 33.7185) (end 71.3105 60.706) (width 0.75) (layer F.Cu) (net 13))
   (segment (start 71.3105 60.706) (end 68.707 63.3095) (width 0.75) (layer F.Cu) (net 13))
   (segment (start 68.707 63.3095) (end 64.6105 63.3095) (width 0.75) (layer F.Cu) (net 13))
-  (segment (start 69.912 32.32) (end 65.49 32.32) (width 0.75) (layer F.Cu) (net 13) (status 800000))
+  (segment (start 69.912 32.32) (end 65.49 32.32) (width 0.75) (layer F.Cu) (net 13))
   (segment (start 63.627 63.3095) (end 64.6105 63.3095) (width 0.75) (layer F.Cu) (net 13))
   (segment (start 62.67 64.2665) (end 63.627 63.3095) (width 0.75) (layer F.Cu) (net 13))
@@
   (segment (start 58.9 31.3) (end 53.45 31.3) (width 1) (layer F.Cu) (net 13))
   (segment (start 59.9 32.3) (end 58.9 31.3) (width 1) (layer F.Cu) (net 13))
-  (segment (start 65.49 34.86) (end 68.7055 34.86) (width 0.75) (layer F.Cu) (net 14) (status 400000))
-  (segment (start 60.13 63.441) (end 60.13 65.25) (width 0.75) (layer F.Cu) (net 14) (status 800000))
+  (segment (start 65.49 34.86) (end 68.7055 34.86) (width 0.75) (layer F.Cu) (net 14))
+  (segment (start 60.13 63.441) (end 60.13 65.25) (width 0.75) (layer F.Cu) (net 14))
   (segment (start 61.5315 62.0395) (end 60.13 63.441) (width 0.75) (layer F.Cu) (net 14))
   (segment (start 67.5005 62.0395) (end 61.5315 62.0395) (width 0.75) (layer F.Cu) (net 14))
@@
   (segment (start 67.75 68.36) (end 67.84 68.45) (width 0.25) (layer F.Cu) (net 25))
   (zone (net 23) (net_name GND) (layer F.Cu) (hatch edge 0.508)
-    (connect_pads (clearance 0.7))
-    (min_thickness 0.3)
+    (connect_pads yes (clearance 0.6))
+    (min_thickness 0.5)
     (fill yes (arc_segments 16) (thermal_gap 0.508) (thermal_bridge_width 0.508) (smoothing chamfer))
     (polygon
@@
   (zone (net 2) (net_name +3V3) (layer F.Cu) (hatch edge 0.508)
     (priority 1)
-    (connect_pads (clearance 0.7))
+    (connect_pads yes (clearance 0.75))
     (min_thickness 0.3)
     (fill yes (arc_segments 16) (thermal_gap 0.508) (thermal_bridge_width 0.508) (smoothing chamfer))
     (polygon
       (pts
-        (xy 24.13 48.26) (xy 26.035 50.165) (xy 24.13 52.07)
+        (xy 40 46) (xy 40.25 46.25) (xy 40.25 49.75) (xy 38.5 51.5) (xy 24.7 51.5)
+        (xy 24.13 52.07) (xy 24.13 48.26) (xy 24.56 48.69) (xy 24.75 48.5) (xy 32.75 48.5)
+        (xy 36.75 44.5) (xy 40 44.5)
       )
     )
+  )
+  (zone (net 0) (net_name "") (layer F.Cu) (hatch edge 0.508)
+    (connect_pads yes (clearance 0.8))
+    (min_thickness 0.4)
+    (keepout (tracks allowed) (vias not_allowed) (copperpour not_allowed))
+    (fill (arc_segments 16) (thermal_gap 0.508) (thermal_bridge_width 0.508))
+    (polygon
+      (pts
+        (xy 52.75 45.75) (xy 40.25 45.75) (xy 40.25 30.5) (xy 52.75 30.5)
+      )
+    )
